File: kicad/Vikingboard.kicad_sch (KiCad schematic)
At the start: 9 parts, among them J1 Conn_02x09_Odd_Even, J2 Conn_02x18_Odd_Even, U1 Conn_01x05, U2 DRV2605LDGS, U3 PAL24, U4 Q_Triac, U5 SX1276, U6 Conn_02x04_Odd_Even_Shielded, U7 Conn_01x08_Shielded

Commit message: Apply prototype net spec to PCB - all 69 nets assigned
Parts:
- J1, J2, U1, U3, U4, U6, U7: footprint (none) -> Connector_PinHeader_2.54mm:PinHeader_1x08_P2.54mm_Vertical
- U2: footprint Package_SO:VSSOP-10_3x3mm_P0.5mm -> Connector_PinHeader_2.54mm:PinHeader_1x08_P2.54mm_Vertical
- U5: footprint Package_DFN_QFN:QFN-28-1EP_6x6mm_P0.65mm_EP4.8x4.8mm -> Connector_PinHeader_2.54mm:PinHeader_1x08_P2.54mm_Vertical
Changed lines of the file:
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@@
 			)
 		)
-		(property "Footprint" ""
+		(property "Footprint" "Connector_PinHeader_2.54mm:PinHeader_1x08_P2.54mm_Vertical"
 			(at -190.5 15.24 0)
 			(effects
@@
 			)
 		)
-		(property "Footprint" ""
+		(property "Footprint" "Connector_PinHeader_2.54mm:PinHeader_1x08_P2.54mm_Vertical"
 			(at -433.07 389.89 0)
 			(effects
@@
 			)
 		)
-		(property "Footprint" ""
+		(property "Footprint" "Connector_PinHeader_2.54mm:PinHeader_1x08_P2.54mm_Vertical"
 			(at -431.8 320.04 0)
 			(effects
@@
 			)
 		)
-		(property "Footprint" ""
+		(property "Footprint" "Connector_PinHeader_2.54mm:PinHeader_1x08_P2.54mm_Vertical"
 			(at -329.565 -51.435 90)
 			(effects
@@
 			)
 		)
-		(property "Footprint" ""
+		(property "Footprint" "Connector_PinHeader_2.54mm:PinHeader_1x08_P2.54mm_Vertical"
 			(at -316.23 374.65 0)
 			(effects
@@
 			)
 		)
-		(property "Footprint" "Package_DFN_QFN:QFN-28-1EP_6x6mm_P0.65mm_EP4.8x4.8mm"
+		(property "Footprint" "Connector_PinHeader_2.54mm:PinHeader_1x08_P2.54mm_Vertical"
 			(at -328.93 29.21 0)
 			(effects
@@
 			)
 		)
-		(property "Footprint" ""
+		(property "Footprint" "Connector_PinHeader_2.54mm:PinHeader_1x08_P2.54mm_Vertical"
 			(at -509.27 389.89 0)
 			(effects
@@
 			)
 		)
-		(property "Footprint" ""
+		(property "Footprint" "Connector_PinHeader_2.54mm:PinHeader_1x08_P2.54mm_Vertical"
 			(at -313.69 203.2 0)
 			(effects
@@
 			)
 		)
-		(property "Footprint" "Package_SO:VSSOP-10_3x3mm_P0.5mm"
+		(property "Footprint" "Connector_PinHeader_2.54mm:PinHeader_1x08_P2.54mm_Vertical"
 			(at -435.61 455.93 0)
 			(effects

Commit message: Add datasheet directory structure and ESP32 datasheets (Issue #5)
- Created organized folder structure under docs/datasheets/
- Moved ESP32-WROOM-32E datasheet to MCU folder
- Moved ESP32 Hardware Design Guidelines to MCU folder
- Added README with download checklist and status tracking
- Added .gitkeep files to preserve empty directories
- Updated generated documentation (vikingboard_98pin_pinout.md)
Parts:
- removed J1: Conn_02x09_Odd_Even, Connector_PinHeader_2.54mm:PinHeader_1x08_P2.54mm_Vertical, symbol Connector_Generic:Conn_02x09_Odd_Even
- removed J2: Conn_02x18_Odd_Even, Connector_PinHeader_2.54mm:PinHeader_1x08_P2.54mm_Vertical, symbol Connector_Generic:Conn_02x18_Odd_Even
- removed U1: Conn_01x05, Connector_PinHeader_2.54mm:PinHeader_1x08_P2.54mm_Vertical, symbol Connector_Generic:Conn_01x05
- removed U2: DRV2605LDGS, Connector_PinHeader_2.54mm:PinHeader_1x08_P2.54mm_Vertical, symbol Driver_Haptic:DRV2605LDGS
- removed U3: PAL24, Connector_PinHeader_2.54mm:PinHeader_1x08_P2.54mm_Vertical, symbol Logic_Programmable:PAL24
- removed U4: Q_Triac, Connector_PinHeader_2.54mm:PinHeader_1x08_P2.54mm_Vertical, symbol Device:Q_Triac
- removed U5: SX1276, Connector_PinHeader_2.54mm:PinHeader_1x08_P2.54mm_Vertical, symbol RF:SX1276
- removed U6: Conn_02x04_Odd_Even_Shielded, Connector_PinHeader_2.54mm:PinHeader_1x08_P2.54mm_Vertical, symbol Connector_Generic_Shielded:Conn_02x04_Odd_Even_Shielded
- removed U7: Conn_01x08_Shielded, Connector_PinHeader_2.54mm:PinHeader_1x08_P2.54mm_Vertical, symbol Connector_Generic_Shielded:Conn_01x08_Shielded
- added C1, C2, C4: 10µF, Capacitor_SMD:C_0805_2012Metric, symbol Device:C
- added C3, C5: 100nF, Capacitor_SMD:C_0805_2012Metric, symbol Device:C
- added J1: VIKINGBOARD_98PIN, vikingboard:EDGE_CONNECTOR_98PIN, symbol vikingboard_connector:VIKINGBOARD_98PIN
- added U1: AMS1117-3.3, Package_TO_SOT_SMD:SOT-223, symbol vikingboard_components:AMS1117-3.3
- added U2: XC6206P332MR, Package_TO_SOT_SMD:SOT-23-3, symbol vikingboard_components:XC6206P332MR
- added U3: IP2721, Package_DFN_QFN:QFN-10, symbol vikingboard_components:IP2721
Other:
- note added: "98-PIN CONNECTOR"
- note added: "POWER SECTION"
- note added: "Power Budget: IO_3V3: 346mA / 1.0A RF_3V3: 192mA / 0.3A"
- company: (none) -> VikingBoard Project
- title: (none) -> VikingBoard 98-Pin

Commit message: PCB Update - 2025-12-05 12:30
✅ Production files updated
- Gerbers regenerated
- DRC passed
- Ready for manufacturing

Changes:
  - kicad/vikingboard_gerbers.zip
  - pcb_scripts/vikingboard_bom_jlcpcb.csv
  - pcb_scripts/vikingboard_cpl.csv
Parts:
- renumbered C5 to C?, C1 to C?, C4 to C?, C2 to C?, C3 to C?, J1 to J?, U1 to U?, U3 to U?, U2 to U?
